File: hardware/kicad/weatherStationBoard/weatherStationBoard.kicad_pcb (KiCad board)
At the start: 2 copper layers, 85 x 35 mm, 61 parts, among them J1 USB_C_Receptacle_USB2.0_16P, J3 Conn_01x30_Pin, Q1 S8050, Q2 S8050, U1 ESP-12F, U2 CH340G, U3 BME680, U4 AMS1117-3.3, Y1 Crystal_GND24_Small

Commit message: Gerberfiles and final Case model
Parts:
- moved C1 178.2 mm to (20.9, 10.7)
- moved C10 178.2 mm to (8.06, 12.9)
- moved C11 178.2 mm to (55.0, 20.0)
- moved C12 178.2 mm to (44.4, 13.1)
- moved C13 178.2 mm to (74.5, 6.70)
- moved C14 178.2 mm to (74.5, 13.9)
- moved C15 178.2 mm to (74.5, 4.45)
- moved C16 178.2 mm to (74.5, 23.4)
- moved C17 178.2 mm to (74.5, 27.5)
- moved C18 178.2 mm to (74.5, 25.4)
- moved C2 178.2 mm to (20.9, 12.8)
- moved C3 178.2 mm to (16.6, 23.5)
- moved C4 178.2 mm to (13.3, 26.4)
- moved C5 178.2 mm to (66.5, 9.00)
- moved C6 178.2 mm to (20.9, 8.65)
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Routing:
- net 3V3: track 154.1 -> 152.7 mm
- net 5V: track 104.2 -> 103.4 mm
- net /I2C_SCL: track 55.4 -> 54.6 mm
- net /nRST: track 86.8 -> 86.1 mm
- net Net-(U2-RXD): track 36.1 -> 35.6 mm
Other:
- copper layers 2 -> 4
- board text added: "The diameter of this milling-path should be d=1mm"
- board text removed: "d=1mm"
